File: boards/timemaster/pcb/timemaster.kicad_sch (KiCad schematic)
At the start: 59 parts, among them J1 Conn_02x03_Odd_Even, J2 Conn_Coaxial, J3 Conn_Coaxial, J4 Conn_Coaxial, J5 Conn_Coaxial, U1 SM05B-GHS-TB(LF)(SN), U2 SATA-401-M07S1BY-A, U3 STM32G031G8Ux, U4 SI5340B-D-GM, U5 TPS62231TDRYRQ1, X1 X2C048000L71H-CEHZ

Commit message: timemaster: rev b with larger vias for jlc
Other:
- title: (none) -> Timemaster
Changed lines of the file:
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@@
 	(generator_version "9.0")
 	(paper "A4")
+	(title_block
+		(title "Timemaster")
+		(date "2026-03-10")
+		(rev "B")
+	)
 	(text_box "Local I2C Pullups"
 		(exclude_from_sim no)
